File: 01_Hardware/v00/esp32_node_v00/esp32_node_v00.kicad_pcb (KiCad board)
At the start: 2 copper layers, 70 x 35 mm, 20 parts

Commit message: Actualizo v00, preproyecto
Routing:
- net (no net): vias 0 -> 2
Other:
- outline, holes or cut-outs redrawn
- board text added: "BOTTOM"
- board text added: "Huecos De Montaje"
Changed lines of the file:
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@@
   (general
     (thickness 1.6)
-    (drawings 20)
-    (tracks 0)
+    (drawings 23)
+    (tracks 2)
     (zones 0)
     (modules 20)
@@
     (mod_text_size 1 1)
     (mod_text_width 0.15)
-    (pad_size 1.524 1.524)
-    (pad_drill 0.762)
+    (pad_size 2 2)
+    (pad_drill 2)
     (pad_to_mask_clearance 0)
     (aux_axis_origin 0 0)
     (grid_origin 121.5 61.5)
-    (visible_elements FFF5F767)
+    (visible_elements FFF7F76F)
     (pcbplotparams
       (layerselection 0x010fc_ffffffff)
@@
     )
     (fp_text value Hirose_DF13-02P-1.25DS_1x02_P1.25mm_Horizontal (at 0.62 -2.1 -90) (layer B.Fab)
-      (effects (font (size 1 1) (thickness 0.15)) (justify mirror))
-    )
-    (fp_text user %R (at 0.62 3.8 -90) (layer B.Fab)
       (effects (font (size 1 1) (thickness 0.15)) (justify mirror))
     )
@@
     (fp_line (start 3.2 -1.4) (end 3.2 5) (layer B.CrtYd) (width 0.05))
     (fp_line (start 3.2 5) (end -1.95 5) (layer B.CrtYd) (width 0.05))
+    (fp_text user %R (at 0.62 3.8 -90) (layer B.Fab)
+      (effects (font (size 1 1) (thickness 0.15)) (justify mirror))
+    )
     (pad 2 thru_hole oval (at 1.25 0 90) (size 0.9 1.4) (drill 0.6) (layers *.Cu *.Mask))
     (pad 1 thru_hole roundrect (at 0 0 90) (size 0.9 1.4) (drill 0.6) (layers *.Cu *.Mask) (roundrect_rratio 0.25))
@@
     (fp_text value microSD_HC_Hirose_DM3D-SF (at -0.025 -6.975 90) (layer B.Fab)
       (effects (font (size 1 1) (thickness 0.15)) (justify mirror))
-    )
-    (fp_arc (start 5.475 -5.475) (end 5.475 -5.725) (angle -90) (layer B.Fab) (width 0.1))
-    (fp_arc (start 4.725 -4.425) (end 4.725 -3.925) (angle -90) (layer B.Fab) (width 0.1))
-    (fp_arc (start -5.525 -5.475) (end -5.275 -5.475) (angle -90) (layer B.Fab) (width 0.1))
-    (fp_arc (start -4.775 -4.425) (end -5.275 -4.425) (angle -90) (layer B.Fab) (width 0.1))
-    (fp_arc (start -5.025 -9.575) (end -5.025 -10.075) (angle -90) (layer B.Fab) (width 0.1))
-    (fp_arc (start 4.975 -9.575) (end 5.475 -9.575) (angle -90) (layer B.Fab) (width 0.1))
-    (fp_text user KEEPOUT (at -0.725 4.8 90) (layer Cmts.User)
-      (effects (font (size 0.4 0.4) (thickness 0.06)))
-    )
-    (fp_text user %R (at -0.025 -1.475 90) (layer B.Fab)
-      (effects (font (size 1 1) (thickness 0.1)) (justify mirror))
-    )
-    (fp_text user KEEPOUT (at -0.275 0.525 90) (layer Cmts.User)
-      (effects (font (size 1 1) (thickness 0.1)))
     )
     (fp_line (start 6.435 2.075) (end 6.435 -4.225) (layer B.SilkS) (width 0.12))
@@
     (fp_line (start 0.525 5.725) (end -1.975 5.725) (layer Dwgs.User) (width 0.1))
     (fp_line (start 6.325 5.785) (end 6.435 5.785) (layer B.SilkS) (width 0.12))
+    (fp_arc (start 5.475 -5.475) (end 5.475 -5.725) (angle -90) (layer B.Fab) (width 0.1))
+    (fp_arc (start 4.725 -4.425) (end 4.725 -3.925) (angle -90) (layer B.Fab) (width 0.1))
+    (fp_arc (start -5.525 -5.475) (end -5.275 -5.475) (angle -90) (layer B.Fab) (width 0.1))
+    (fp_arc (start -4.775 -4.425) (end -5.275 -4.425) (angle -90) (layer B.Fab) (width 0.1))
+    (fp_arc (start -5.025 -9.575) (end -5.025 -10.075) (angle -90) (layer B.Fab) (width 0.1))
+    (fp_arc (start 4.975 -9.575) (end 5.475 -9.575) (angle -90) (layer B.Fab) (width 0.1))
+    (fp_text user KEEPOUT (at -0.725 4.8 90) (layer Cmts.User)
+      (effects (font (size 0.4 0.4) (thickness 0.06)))
+    )
+    (fp_text user %R (at -0.025 -1.475 90) (layer B.Fab)
+      (effects (font (size 1 1) (thickness 0.1)) (justify mirror))
+    )
+    (fp_text user KEEPOUT (at -0.275 0.525 90) (layer Cmts.User)
+      (effects (font (size 1 1) (thickness 0.1)))
+    )
     (pad 10 smd rect (at 5.575 5.45 270) (size 1 1.55) (layers B.Cu B.Paste B.Mask))
     (pad 11 smd rect (at 5.625 -5.225 270) (size 1.5 1.5) (layers B.Cu B.Paste B.Mask))
@@
       (effects (font (size 1 1) (thickness 0.15)))
     )
-    (fp_text user %R (at 0 -3.75) (layer F.Fab)
-      (effects (font (size 1 1) (thickness 0.15)))
-    )
     (fp_line (start 3.2 2.1) (end 3.2 1.6) (layer F.Fab) (width 0.1))
     (fp_line (start 3.2 -2.1) (end 3.2 -1.6) (layer F.Fab) (width 0.1))
@@
     (fp_line (start -4.25 3) (end -4.25 -3) (layer F.CrtYd) (width 0.05))
     (fp_circle (center 0 0) (end 1 0) (layer F.Fab) (width 0.1))
+    (fp_text user %R (at 0 -3.75) (layer F.Fab)
+      (effects (font (size 1 1) (thickness 0.15)))
+    )
     (pad 2 smd rect (at 3.15 1.9) (size 1.7 1) (layers F.Cu F.Paste F.Mask))
     (pad 2 smd rect (at -3.15 1.9) (size 1.7 1) (layers F.Cu F.Paste F.Mask))
@@
     )
     (fp_text value SMA_Amphenol_132289_EdgeMount (at 5 -6) (layer B.Fab)
-      (effects (font (size 1 1) (thickness 0.15)) (justify mirror))
-    )
-    (fp_text user %R (at 4.79 0 -90) (layer B.Fab)
       (effects (font (size 1 1) (thickness 0.15)) (justify mirror))
     )
@@
     (fp_line (start -1.91 -3.81) (end -1.91 -5.08) (layer B.Fab) (width 0.1))
     (fp_line (start -1.91 -5.08) (end 4.445 -5.08) (layer B.Fab) (width 0.1))
+    (fp_text user %R (at 4.79 0 -90) (layer B.Fab)
+      (effects (font (size 1 1) (thickness 0.15)) (justify mirror))
+    )
     (pad 1 smd rect (at 0 0 270) (size 1.5 5.08) (layers B.Cu B.Paste B.Mask))
     (pad 2 smd rect (at 0 4.25 270) (size 1.5 5.08) (layers B.Cu B.Paste B.Mask))
@@
       (effects (font (size 1 1) (thickness 0.15)))
     )
-    (fp_text user %R (at 0 3.5) (layer F.Fab)
-      (effects (font (size 1 1) (thickness 0.15)))
-    )
     (fp_line (start 0 1) (end 0.3 1.3) (layer F.Fab) (width 0.1))
     (fp_line (start -0.3 1.3) (end 0 1) (layer F.Fab) (width 0.1))
@@
     (fp_line (start -1 1.3) (end 1.3 1.3) (layer F.Fab) (width 0.1))
     (fp_circle (center 0 0) (end 0 0.2) (layer F.Fab) (width 0.1))
+    (fp_text user %R (at 0 3.5) (layer F.Fab)
+      (effects (font (size 1 1) (thickness 0.15)))
+    )
     (pad 1 smd rect (at 0 1.5) (size 1 1) (layers F.Cu F.Paste F.Mask))
     (pad 2 smd rect (at 0 -1.5) (size 1 1) (layers F.Cu F.Paste F.Mask))
@@
     )
   )
+  (gr_text BOTTOM (at 149.5 68.5) (layer F.SilkS)
+    (effects (font (size 6 6) (thickness 1) italic) (justify mirror))
+  )
+  (gr_text "Huecos\nDe\nMontaje" (at 171.5 95.5) (layer F.SilkS)
+    (effects (font (size 0.5 0.5) (thickness 0.125)))
+  )
+  (gr_text "Huecos\nDe\nMontaje" (at 142.5 95.5) (layer F.SilkS)
+    (effects (font (size 0.5 0.5) (thickness 0.125)))
+  )
   (gr_line (start 114 110.5) (end 180 110.5) (layer Edge.Cuts) (width 0.05))
   (gr_line (start 180 75.5) (end 114 75.5) (layer Edge.Cuts) (width 0.05))
-  (dimension 70 (width 0.15) (layer F.Fab)
-    (gr_text "70,000 mm" (at 147 116.3) (layer F.Fab)
-      (effects (font (size 1 1) (thickness 0.15)))
+  (dimension 70 (width 0.15) (layer F.SilkS)
+    (gr_text "70,000 mm" (at 147 116.3) (layer F.SilkS)
+      (effects (font (size 1 1) (thickness 0.15)) (justify mirror))
     )
     (feature1 (pts (xy 182 115) (xy 182 115.586421)))
@@
     (arrow2b (pts (xy 112 115) (xy 113.126504 114.413579)))
   )
-  (gr_line (start 151 99.5) (end 151 97.5) (layer Edge.Cuts) (width 0.05))
-  (gr_line (start 164 97.5) (end 164 99.5) (layer Edge.Cuts) (width 0.05))
-  (gr_line (start 151 97.5) (end 157.5 97.5) (layer Edge.Cuts) (width 0.05))
-  (gr_line (start 164 97.5) (end 157.5 97.5) (layer Edge.Cuts) (width 0.05))
-  (gr_line (start 151 99.5) (end 157.5 99.5) (layer Edge.Cuts) (width 0.05))
-  (gr_line (start 164 99.5) (end 157.5 99.5) (layer Edge.Cuts) (width 0.05))
+  (gr_line (start 148.5 99.5) (end 148.5 97.5) (layer Edge.Cuts) (width 0.05))
+  (gr_line (start 166.5 97.5) (end 166.5 99.5) (layer Edge.Cuts) (width 0.05))
+  (gr_line (start 148.5 97.5) (end 157.5 97.5) (layer Edge.Cuts) (width 0.05))
+  (gr_line (start 166.5 97.5) (end 157.5 97.5) (layer Edge.Cuts) (width 0.05))
+  (gr_line (start 148.5 99.5) (end 157.5 99.5) (layer Edge.Cuts) (width 0.05))
+  (gr_line (start 166.5 99.5) (end 157.5 99.5) (layer Edge.Cuts) (width 0.05))
   (gr_line (start 182 77.5) (end 182 108.5) (layer Edge.Cuts) (width 0.05))
   (gr_line (start 180 75.5) (end 182 77.5) (layer Edge.Cuts) (width 0.05))
@@
   (gr_line (start 112 86) (end 112 77.5) (layer Edge.Cuts) (width 0.05))
   (gr_line (start 114 75.5) (end 112 77.5) (layer Edge.Cuts) (width 0.05))
-  (dimension 35 (width 0.15) (layer Dwgs.User)
-    (gr_text "35,000 mm" (at 107.8 93 90) (layer Dwgs.User)
-      (effects (font (size 1 1) (thickness 0.15)))
+  (dimension 35 (width 0.15) (layer F.SilkS)
+    (gr_text "35,000 mm" (at 107.8 93 90) (layer F.SilkS)
+      (effects (font (size 1 1) (thickness 0.15)) (justify mirror))
     )
     (feature1 (pts (xy 106.5 75.5) (xy 107.086421 75.5)))
@@
   (gr_line (start 114 110.5) (end 112 108.5) (layer Edge.Cuts) (width 0.05))
   (gr_line (start 114 98) (end 112 100) (layer Edge.Cuts) (width 0.05))
+  (via (at 144.5 92.5) (size 2.1) (drill 2) (layers F.Cu B.Cu) (net 0))
+  (via (at 170.5 92.5) (size 2.1) (drill 2) (layers F.Cu B.Cu) (net 0))
 )
